Commit message: added ros_control tag to urdf, will focus on the fact that this breaks simulation later

File: ros/src/leremix_description/urdf/LeRemix.xacro (robot description, xacro)
@@ -1221,3 +1221,58 @@
   <child link="upper_floor_1"/>
 </joint>
+<!-- ros2_control hardware interface -->
+<ros2_control name="leremix_hardware" type="system">
+  <hardware>
+    <plugin>leremix_control_plugin/Esp32SystemTopic</plugin>
+    <param name="base_cmd_topic">/esp32/base_cmd</param>
+    <param name="arm_cmd_topic">/esp32/arm_cmd</param>
+    <param name="state_topic">/esp32/joint_states</param>
+    <param name="publish_if_unchanged">true</param>
+  </hardware>
+  <!-- Base joints - velocity command, position+velocity states -->
+  <joint name="back_motor_rotation">
+    <command_interface name="velocity"/>
+    <state_interface name="position"/>
+    <state_interface name="velocity"/>
+  </joint>
+  <joint name="left_motor_rotation">
+    <command_interface name="velocity"/>
+    <state_interface name="position"/>
+    <state_interface name="velocity"/>
+  </joint>
+  <joint name="right_motor_rotation">
+    <command_interface name="velocity"/>
+    <state_interface name="position"/>
+    <state_interface name="velocity"/>
+  </joint>
+  <!-- Arm joints - position command, position state -->
+  <joint name="1">
+    <command_interface name="position"/>
+    <state_interface name="position"/>
+  </joint>
+  <joint name="2">
+    <command_interface name="position"/>
+    <state_interface name="position"/>
+  </joint>
+  <joint name="3">
+    <command_interface name="position"/>
+    <state_interface name="position"/>
+  </joint>
+  <joint name="4">
+    <command_interface name="position"/>
+    <state_interface name="position"/>
+  </joint>
+  <joint name="5">
+    <command_interface name="position"/>
+    <state_interface name="position"/>
+  </joint>
+  <joint name="6">
+    <command_interface name="position"/>
+    <state_interface name="position"/>
+  </joint>
+  <joint name="camera_tilt">
+    <command_interface name="position"/>
+    <state_interface name="position"/>
+  </joint>
+</ros2_control>
 </robot>

Commit message: adding tower, bastardized URDF

File: ros/src/leremix_description/urdf/LeRemix.xacro (robot description, xacro)
@@ -4,87 +4,19 @@
 <link name="base_link">
   <inertial>
-    <origin xyz="-0.0062553486303642105 3.340802284881761e-05 0.0025000000000011367" rpy="0 0 0"/>
-    <mass value="0.6"/>
-    <inertia ixx="0.002" iyy="0.0019" izz="0.004" ixy="-2e-06" iyz="0.0" ixz="0.0"/>
+    <origin xyz="-0.006995872672132321 0.00016351719531705557 -0.0020614117608215563" rpy="0 0 0"/>
+    <mass value="1.5793453539076083"/>
+    <inertia ixx="0.00541" iyy="0.005179" izz="0.010582" ixy="-3e-06" iyz="0.0" ixz="0.0"/>
   </inertial>
   <visual>
     <origin xyz="0 0 0" rpy="0 0 0"/>
     <geometry>
-      <mesh filename="file://$(find leremix_description)/meshes/base_link.stl" scale="0.001 0.001 0.001"/>
-    </geometry>
-    <material name="darkgray"/>
+      <mesh filename="file://$(find LeRemix_description)/meshes/base_link.stl" scale="0.001 0.001 0.001"/>
+    </geometry>
+    <material name="silver"/>
   </visual>
   <collision>
     <origin xyz="0 0 0" rpy="0 0 0"/>
     <geometry>
-      <mesh filename="file://$(find leremix_description)/meshes/base_link.stl" scale="0.001 0.001 0.001"/>
-    </geometry>
-  </collision>
-</link>
-<link name="back_wheel_1">
-  <inertial>
-    <origin xyz="-0.015374630356382424 -4.805049047319634e-07 4.6137978126914447e-07" rpy="0 0 0"/>
-    <mass value="0.32"/>
-    <inertia ixx="0.00045" iyy="0.00026" izz="0.00026" ixy="0.0" iyz="0.0" ixz="0.0"/>
-  </inertial>
-  <visual>
-    <origin xyz="0.11523 -7e-06 -0.015198" rpy="0 0 0"/>
-    <geometry>
-      <mesh filename="file://$(find leremix_description)/meshes/back_wheel_1.stl" scale="0.001 0.001 0.001"/>
-    </geometry>
-    <material name="darkgray"/>
-  </visual>
-<collision>
-  <!-- roll=0, pitch=+90°, yaw=180° -->
-  <origin xyz="0 0 0" rpy="0 1.57079632679 3.14159265359"/>
-  <geometry>
-      <cylinder radius="0.05" length="0.04"/>
-  </geometry>
-</collision>
-</link>
-<link name="right_wheel_1">
-  <inertial>
-    <origin xyz="0.007687514715893053 -0.01331534843579213 3.7606430000614033e-07" rpy="0 0 0"/>
-    <mass value="0.32"/>
-    <inertia ixx="0.00031" iyy="0.0004" izz="0.00026" ixy="-8e-05" iyz="0.0" ixz="0.0"/>
-  </inertial>
-  <visual>
-    <origin xyz="-0.057621 0.099788 -0.015217" rpy="0 0 0"/>
-    <geometry>
-      <mesh filename="file://$(find leremix_description)/meshes/right_wheel_1.stl" scale="0.001 0.001 0.001"/>
-    </geometry>
-    <material name="darkgray"/>
-  </visual>
- <collision>
-  <!-- roll=0, pitch=+90°, yaw=120° -->
-  <origin xyz="0 0 0" rpy="0 1.57079632679 2.09439510239"/>
-  <geometry>
-      <cylinder radius="0.05" length="0.04"/>
-  </geometry>
-</collision>
-</link>
-<link name="left_wheel_1">
-  <inertial>
-    <origin xyz="0.007687890146983539 0.013314999193957927 1.1659539730229929e-07" rpy="0 0 0"/>
-    <mass value="0.32"/>
-    <inertia ixx="0.00031" iyy="0.0004" izz="0.00026" ixy="8e-05" iyz="0.0" ixz="0.0"/>
-  </inertial>
-  <visual>
-    <origin xyz="-0.057571 -0.099817 -0.015181" rpy="0 0 0"/>
-    <geometry>
-      <mesh filename="file://$(find leremix_description)/meshes/left_wheel_1.stl" scale="0.001 0.001 0.001"/>
-    </geometry>
-    <material name="darkgray"/>
-  </visual>
-  <!--<collision>
-    <origin xyz="-0.057571 -0.099817 -0.015181" rpy="0 0 0"/>
-    <geometry>
-      <mesh filename="file://$(find leremix_description)/meshes/left_wheel_1.stl" scale="0.001 0.001 0.001"/>
-    </geometry>
-  </collision>-->
-  <collision>
-    <origin xyz="0 0 0" rpy="0 1.57079632679 -2.09439510239"/>
-    <geometry>
-      <cylinder radius="0.05" length="0.04"/>
+      <mesh filename="file://$(find LeRemix_description)/meshes/base_link.stl" scale="0.001 0.001 0.001"/>
     </geometry>
   </collision>
@@ -92,19 +24,19 @@
 <link name="arm_base_rotation_servo_1">
   <inertial>
-    <origin xyz="0.019999032189425586 0.010249751352693647 0.01602706492472336" rpy="0 0 0"/>
-    <mass value="0.025"/>
-    <inertia ixx="3.6e-06" iyy="6.8e-06" izz="5.4e-06" ixy="0.0" iyz="0.0" ixz="0.0"/>
-  </inertial>
-  <visual>
-    <origin xyz="-0.044348 0.01025 -0.0853" rpy="0 0 0"/>
-    <geometry>
-      <mesh filename="file://$(find leremix_description)/meshes/arm_base_rotation_servo_1.stl" scale="0.001 0.001 0.001"/>
-    </geometry>
-    <material name="darkgray"/>
-  </visual>
-  <collision>
-    <origin xyz="-0.044348 0.01025 -0.0853" rpy="0 0 0"/>
-    <geometry>
-      <mesh filename="file://$(find leremix_description)/meshes/arm_base_rotation_servo_1.stl" scale="0.001 0.001 0.001"/>
+    <origin xyz="0.019999508147657045 0.010249860525163957 0.01602665316389948" rpy="0 0 0"/>
+    <mass value="0.2843033831904074"/>
+    <inertia ixx="4e-05" iyy="7.3e-05" izz="6.2e-05" ixy="0.0" iyz="0.0" ixz="-1e-06"/>
+  </inertial>
+  <visual>
+    <origin xyz="-0.043607 0.01012 -0.080739" rpy="0 0 0"/>
+    <geometry>
+      <mesh filename="file://$(find LeRemix_description)/meshes/arm_base_rotation_servo_1.stl" scale="0.001 0.001 0.001"/>
+    </geometry>
+    <material name="silver"/>
+  </visual>
+  <collision>
+    <origin xyz="-0.043607 0.01012 -0.080739" rpy="0 0 0"/>
+    <geometry>
+      <mesh filename="file://$(find LeRemix_description)/meshes/arm_base_rotation_servo_1.stl" scale="0.001 0.001 0.001"/>
     </geometry>
   </collision>
@@ -112,19 +44,19 @@
 <link name="arm_shoulder_link_1">
   <inertial>
-    <origin xyz="-0.05594320151702218 0.019699275433957473 -0.015368254886761495" rpy="0 0 0"/>
-    <mass value="0.09"/>
-    <inertia ixx="5.1e-05" iyy="0.000113" izz="0.00014" ixy="-8e-07" iyz="0.0" ixz="-2.7e-05"/>
-  </inertial>
-  <visual>
-    <origin xyz="-0.107748 0.0183 -0.1741" rpy="0 0 0"/>
-    <geometry>
-      <mesh filename="file://$(find leremix_description)/meshes/arm_shoulder_link_1.stl" scale="0.001 0.001 0.001"/>
-    </geometry>
-    <material name="darkgray"/>
-  </visual>
-  <collision>
-    <origin xyz="-0.107748 0.0183 -0.1741" rpy="0 0 0"/>
-    <geometry>
-      <mesh filename="file://$(find leremix_description)/meshes/arm_shoulder_link_1.stl" scale="0.001 0.001 0.001"/>
+    <origin xyz="-0.05439041310030922 0.019699384606440277 -0.020185957481023337" rpy="0 0 0"/>
+    <mass value="0.9906249126045027"/>
+    <inertia ixx="0.000624" iyy="0.001251" izz="0.001489" ixy="-7e-06" iyz="-3e-06" ixz="-0.000385"/>
+  </inertial>
+  <visual>
+    <origin xyz="-0.107007 0.01817 -0.169539" rpy="0 0 0"/>
+    <geometry>
+      <mesh filename="file://$(find LeRemix_description)/meshes/arm_shoulder_link_1.stl" scale="0.001 0.001 0.001"/>
+    </geometry>
+    <material name="silver"/>
+  </visual>
+  <collision>
+    <origin xyz="-0.107007 0.01817 -0.169539" rpy="0 0 0"/>
+    <geometry>
+      <mesh filename="file://$(find LeRemix_description)/meshes/arm_shoulder_link_1.stl" scale="0.001 0.001 0.001"/>
     </geometry>
   </collision>
@@ -132,19 +64,19 @@
 <link name="arm_elbow_servo_1">
   <inertial>
-    <origin xyz="-0.015077042423432949 -0.016027313578791422 0.016664878981827835" rpy="0 0 0"/>
-    <mass value="0.025"/>
-    <inertia ixx="6.3e-06" iyy="5.4e-06" izz="3.6e-06" ixy="0.0" iyz="0.0" ixz="1e-06"/>
-  </inertial>
-  <visual>
-    <origin xyz="-0.010157 -0.0178 -0.142981" rpy="0 0 0"/>
-    <geometry>
-      <mesh filename="file://$(find leremix_description)/meshes/arm_elbow_servo_1.stl" scale="0.001 0.001 0.001"/>
-    </geometry>
-    <material name="darkgray"/>
-  </visual>
-  <collision>
-    <origin xyz="-0.010157 -0.0178 -0.142981" rpy="0 0 0"/>
-    <geometry>
-      <mesh filename="file://$(find leremix_description)/meshes/arm_elbow_servo_1.stl" scale="0.001 0.001 0.001"/>
+    <origin xyz="-0.016472070877660654 -0.016027204406308133 0.015286802190772275" rpy="0 0 0"/>
+    <mass value="0.2843033831904074"/>
+    <inertia ixx="7e-05" iyy="6.2e-05" izz="4.4e-05" ixy="-0.0" iyz="1e-06" ixz="1.1e-05"/>
+  </inertial>
+  <visual>
+    <origin xyz="-0.0125 -0.01793 -0.130033" rpy="0 0 0"/>
+    <geometry>
+      <mesh filename="file://$(find LeRemix_description)/meshes/arm_elbow_servo_1.stl" scale="0.001 0.001 0.001"/>
+    </geometry>
+    <material name="silver"/>
+  </visual>
+  <collision>
+    <origin xyz="-0.0125 -0.01793 -0.130033" rpy="0 0 0"/>
+    <geometry>
+      <mesh filename="file://$(find LeRemix_description)/meshes/arm_elbow_servo_1.stl" scale="0.001 0.001 0.001"/>
     </geometry>
   </collision>
@@ -152,19 +84,19 @@
 <link name="arm_elbow_link_1">
   <inertial>
-    <origin xyz="-0.010924420778980003 0.015214630153971578 0.06115198501523547" rpy="0 0 0"/>
-    <mass value="0.075"/>
-    <inertia ixx="0.0001" iyy="8.2e-05" izz="3.2e-05" ixy="1.5e-06" iyz="-1e-05" ixz="1.3e-05"/>
-  </inertial>
-  <visual>
-    <origin xyz="0.008233 0.0168 -0.172011" rpy="0 0 0"/>
-    <geometry>
-      <mesh filename="file://$(find leremix_description)/meshes/arm_elbow_link_1.stl" scale="0.001 0.001 0.001"/>
-    </geometry>
-    <material name="darkgray"/>
-  </visual>
-  <collision>
-    <origin xyz="0.008233 0.0168 -0.172011" rpy="0 0 0"/>
-    <geometry>
-      <mesh filename="file://$(find leremix_description)/meshes/arm_elbow_link_1.stl" scale="0.001 0.001 0.001"/>
+    <origin xyz="0.05832603889171534 0.015214739326452977 0.021377048894272332" rpy="0 0 0"/>
+    <mass value="0.8772447501056027"/>
+    <inertia ixx="0.000473" iyy="0.000993" izz="0.001135" ixy="-0.000109" iyz="-4.1e-05" ixz="-0.000289"/>
+  </inertial>
+  <visual>
+    <origin xyz="0.00835 0.01667 -0.157349" rpy="0 0 0"/>
+    <geometry>
+      <mesh filename="file://$(find LeRemix_description)/meshes/arm_elbow_link_1.stl" scale="0.001 0.001 0.001"/>
+    </geometry>
+    <material name="silver"/>
+  </visual>
+  <collision>
+    <origin xyz="0.00835 0.01667 -0.157349" rpy="0 0 0"/>
+    <geometry>
+      <mesh filename="file://$(find LeRemix_description)/meshes/arm_elbow_link_1.stl" scale="0.001 0.001 0.001"/>
     </geometry>
   </collision>
@@ -172,19 +104,19 @@
 <link name="arm_wrist_tilt_servo_1">
   <inertial>
-    <origin xyz="0.008468412947984283 -0.0160273135787885 0.020816572929282573" rpy="0 0 0"/>
-    <mass value="0.025"/>
-    <inertia ixx="7.3e-05" iyy="6.2e-05" izz="4e-05" ixy="-0.0" iyz="1e-06" ixz="3e-06"/>
-  </inertial>
-  <visual>
-    <origin xyz="0.041352 -0.0193 -0.270861" rpy="0 0 0"/>
-    <geometry>
-      <mesh filename="file://$(find leremix_description)/meshes/arm_wrist_tilt_servo_1.stl" scale="0.001 0.001 0.001"/>
-    </geometry>
-    <material name="darkgray"/>
-  </visual>
-  <collision>
-    <origin xyz="0.041352 -0.0193 -0.270861" rpy="0 0 0"/>
-    <geometry>
-      <mesh filename="file://$(find leremix_description)/meshes/arm_wrist_tilt_servo_1.stl" scale="0.001 0.001 0.001"/>
+    <origin xyz="0.02197013497411679 -0.016027204406307824 -0.004724364582700924" rpy="0 0 0"/>
+    <mass value="0.2843033831904074"/>
+    <inertia ixx="4.2e-05" iyy="6.2e-05" izz="7.1e-05" ixy="1e-06" iyz="0.0" ixz="-8e-06"/>
+  </inertial>
+  <visual>
+    <origin xyz="-0.083248 -0.01943 -0.207129" rpy="0 0 0"/>
+    <geometry>
+      <mesh filename="file://$(find LeRemix_description)/meshes/arm_wrist_tilt_servo_1.stl" scale="0.001 0.001 0.001"/>
+    </geometry>
+    <material name="silver"/>
+  </visual>
+  <collision>
+    <origin xyz="-0.083248 -0.01943 -0.207129" rpy="0 0 0"/>
+    <geometry>
+      <mesh filename="file://$(find LeRemix_description)/meshes/arm_wrist_tilt_servo_1.stl" scale="0.001 0.001 0.001"/>
     </geometry>
   </collision>
@@ -192,19 +124,19 @@
 <link name="arm_wrist_link_1">
   <inertial>
-    <origin xyz="0.020365813342817646 0.016809532618007075 0.01676666541103805" rpy="0 0 0"/>
-    <mass value="0.045"/>
-    <inertia ixx="2.9e-05" iyy="2.2e-05" izz="3.2e-05" ixy="8e-07" iyz="8e-07" ixz="-7e-06"/>
-  </inertial>
-  <visual>
-    <origin xyz="0.033999 0.0153 -0.30443" rpy="0 0 0"/>
-    <geometry>
-      <mesh filename="file://$(find leremix_description)/meshes/arm_wrist_link_1.stl" scale="0.001 0.001 0.001"/>
-    </geometry>
-    <material name="darkgray"/>
-  </visual>
-  <collision>
-    <origin xyz="0.033999 0.0153 -0.30443" rpy="0 0 0"/>
-    <geometry>
-      <mesh filename="file://$(find leremix_description)/meshes/arm_wrist_link_1.stl" scale="0.001 0.001 0.001"/>
+    <origin xyz="0.02004856305995592 0.01680964179048719 -0.017145371524283942" rpy="0 0 0"/>
+    <mass value="0.2392168278135931"/>
+    <inertia ixx="0.000157" iyy="0.000115" izz="0.000169" ixy="5e-06" iyz="-4e-06" ixz="3.6e-05"/>
+  </inertial>
+  <visual>
+    <origin xyz="-0.117583 0.01517 -0.205718" rpy="0 0 0"/>
+    <geometry>
+      <mesh filename="file://$(find LeRemix_description)/meshes/arm_wrist_link_1.stl" scale="0.001 0.001 0.001"/>
+    </geometry>
+    <material name="silver"/>
+  </visual>
+  <collision>
+    <origin xyz="-0.117583 0.01517 -0.205718" rpy="0 0 0"/>
+    <geometry>
+      <mesh filename="file://$(find LeRemix_description)/meshes/arm_wrist_link_1.stl" scale="0.001 0.001 0.001"/>
     </geometry>
   </collision>
@@ -212,19 +144,19 @@
 <link name="arm_wrist_roll_servo_1">
   <inertial>
-    <origin xyz="-0.00542485104955742 0.01599805621315295 -0.017781280256448873" rpy="0 0 0"/>
-    <mass value="0.025"/>
-    <inertia ixx="6.5e-05" iyy="3.8e-05" izz="6.7e-05" ixy="-1e-06" iyz="-1e-06" ixz="-5e-06"/>
-  </inertial>
-  <visual>
-    <origin xyz="-0.004408 0.0242 -0.349472" rpy="0 0 0"/>
-    <geometry>
-      <mesh filename="file://$(find leremix_description)/meshes/arm_wrist_roll_servo_1.stl" scale="0.001 0.001 0.001"/>
-    </geometry>
-    <material name="darkgray"/>
-  </visual>
-  <collision>
-    <origin xyz="-0.004408 0.0242 -0.349472" rpy="0 0 0"/>
-    <geometry>
-      <mesh filename="file://$(find leremix_description)/meshes/arm_wrist_roll_servo_1.stl" scale="0.001 0.001 0.001"/>
+    <origin xyz="-0.018454007185755128 0.01599816538563275 0.002254236765901807" rpy="0 0 0"/>
+    <mass value="0.2799142523131049"/>
+    <inertia ixx="6.5e-05" iyy="3.8e-05" izz="6.7e-05" ixy="-1e-06" iyz="1e-06" ixz="5e-06"/>
+  </inertial>
+  <visual>
+    <origin xyz="-0.168611 0.02407 -0.175716" rpy="0 0 0"/>
+    <geometry>
+      <mesh filename="file://$(find LeRemix_description)/meshes/arm_wrist_roll_servo_1.stl" scale="0.001 0.001 0.001"/>
+    </geometry>
+    <material name="silver"/>
+  </visual>
+  <collision>
+    <origin xyz="-0.168611 0.02407 -0.175716" rpy="0 0 0"/>
+    <geometry>
+      <mesh filename="file://$(find LeRemix_description)/meshes/arm_wrist_roll_servo_1.stl" scale="0.001 0.001 0.001"/>
     </geometry>
   </collision>
@@ -232,19 +164,19 @@
 <link name="arm_gripper_1">
   <inertial>
-    <origin xyz="0.025535001111388626 0.012976471440615246 0.015105596654687414" rpy="0 0 0"/>
-    <mass value="0.06"/>
-    <inertia ixx="2.9e-05" iyy="4.1e-05" izz="3.8e-05" ixy="-7e-06" iyz="-3e-06" ixz="-1e-05"/>
-  </inertial>
-  <visual>
-    <origin xyz="-0.013096 -0.0048 -0.343356" rpy="0 0 0"/>
-    <geometry>
-      <mesh filename="file://$(find leremix_description)/meshes/arm_gripper_1.stl" scale="0.001 0.001 0.001"/>
-    </geometry>
-    <material name="darkgray"/>
-  </visual>
-  <collision>
-    <origin xyz="-0.013096 -0.0048 -0.343356" rpy="0 0 0"/>
-    <geometry>
-      <mesh filename="file://$(find leremix_description)/meshes/arm_gripper_1.stl" scale="0.001 0.001 0.001"/>
+    <origin xyz="0.01931093722742444 0.012976580613095201 -0.02252356144231421" rpy="0 0 0"/>
+    <mass value="0.44698022927880193"/>
+    <inertia ixx="0.000255" iyy="0.000308" izz="0.000237" ixy="-3e-05" iyz="4.4e-05" ixz="8.2e-05"/>
+  </inertial>
+  <visual>
+    <origin xyz="-0.164095 -0.00493 -0.166097" rpy="0 0 0"/>
+    <geometry>
+      <mesh filename="file://$(find LeRemix_description)/meshes/arm_gripper_1.stl" scale="0.001 0.001 0.001"/>
+    </geometry>
+    <material name="silver"/>
+  </visual>
+  <collision>
+    <origin xyz="-0.164095 -0.00493 -0.166097" rpy="0 0 0"/>
+    <geometry>
+      <mesh filename="file://$(find LeRemix_description)/meshes/arm_gripper_1.stl" scale="0.001 0.001 0.001"/>
     </geometry>
   </collision>
@@ -252,19 +184,19 @@
 <link name="arm_gripper_servo_1">
   <inertial>
-    <origin xyz="-0.006350148409992207 -0.012507811253031454 0.023772399666475375" rpy="0 0 0"/>
-    <mass value="0.025"/>
-    <inertia ixx="6.7e-05" iyy="4.3e-05" izz="6.4e-05" ixy="-5e-06" iyz="6e-06" ixz="8e-06"/>
-  </inertial>
-  <visual>
-    <origin xyz="-0.035579 -0.010832 -0.336363" rpy="0 0 0"/>
-    <geometry>
-      <mesh filename="file://$(find leremix_description)/meshes/arm_gripper_servo_1.stl" scale="0.001 0.001 0.001"/>
-    </geometry>
-    <material name="darkgray"/>
-  </visual>
-  <collision>
-    <origin xyz="-0.035579 -0.010832 -0.336363" rpy="0 0 0"/>
-    <geometry>
-      <mesh filename="file://$(find leremix_description)/meshes/arm_gripper_servo_1.stl" scale="0.001 0.001 0.001"/>
+    <origin xyz="0.02230864527990775 -0.012507702080551863 0.010382401144092585" rpy="0 0 0"/>
+    <mass value="0.2843033831904074"/>
+    <inertia ixx="6.7e-05" iyy="4.3e-05" izz="6.5e-05" ixy="5e-06" iyz="6e-06" ixz="-8e-06"/>
+  </inertial>
+  <visual>
+    <origin xyz="-0.161113 -0.010962 -0.142741" rpy="0 0 0"/>
+    <geometry>
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