Commit message: navigation done

File: ros/src/llmy_description/urdf/LLMy.xacro (robot description, xacro)
@@ -590,7 +590,7 @@
   </visual>
   <collision>
-    <origin xyz="-0.059994 0.089655 -0.017248" rpy="0 0 0"/>
-    <geometry>
-      <mesh filename="file://$(find llmy_description)/meshes/wheel_right_1.stl" scale="0.001 0.001 0.001"/>
+    <origin xyz="0.0 -0.0125 0.0" rpy="1.5708 0 0"/>
+    <geometry>
+      <cylinder radius="0.039" length="0.025"/>
     </geometry>
   </collision>
@@ -610,7 +610,7 @@
   </visual>
   <collision>
-    <origin xyz="-0.059995 -0.089655 -0.017248" rpy="0 0 0"/>
-    <geometry>
-      <mesh filename="file://$(find llmy_description)/meshes/wheel_left_1.stl" scale="0.001 0.001 0.001"/>
+    <origin xyz="0.0 0.0125 0.0" rpy="1.5708 0 0"/>
+    <geometry>
+      <cylinder radius="0.039" length="0.025"/>
     </geometry>
   </collision>
