Commit message: updated with new version

File: ros/src/llmy_control/urdf/LLMy.hardware.xacro (robot description, xacro)
@@ -1,4 +1,6 @@
 <?xml version="1.0"?>
 <robot name="LLMy" xmlns:xacro="http://www.ros.org/wiki/xacro">
+    <!-- Force sim off so LLMy.xacro doesn't include the Gazebo ros2_control block. -->
+    <xacro:arg name="use_sim" default="false"/>
     <!-- Base model from description (without sim ros2_control) -->
     <xacro:include filename="$(find llmy_description)/urdf/LLMy.xacro"/>
@@ -54,9 +56,5 @@
             <state_interface name="velocity"/>
         </joint>
-        <!-- Head/camera joints -->
-        <joint name="pan">
-            <command_interface name="position"/>
-            <state_interface name="position"/>
-        </joint>
+        <!-- Head/camera joint (canvas design: tilt only, no pan) -->
         <joint name="tilt">
             <command_interface name="position"/>

File: ros/src/llmy_description/urdf/LLMy.xacro (robot description, xacro)
@@ -1,1266 +1,1252 @@
 <?xml version="1.0" ?>
+<!--
+  LLMy — URDF for the canvas-design robot, ported into the llmy_root contract
+  so that sibling packages (llmy_control, llmy_moveit, llmy_servo_manager,
+  llmy_slam, llmy_nav, ...) keep working without modification.
+  External names preserved from the original /home/cdr/LLMy llmy_description:
+    joints:  1..6, tilt, right_wheel_joint, left_wheel_joint
+             (pan removed — canvas design has no pan servo)
+    arm links:  arm_base_1, arm_base_rotation_servo_1, arm_base_rotation_link_1,
+                arm_shoulder_servo_1, arm_shoulder_link_1, arm_elbow_servo_1,
+                arm_elbow_link_1, arm_wrist_tilt_servo_1, arm_wrist_link_1,
+                arm_wrist_roll_servo_1, arm_gripper_1, arm_gripper_servo_1, arm_jaw_1
+    sensors:    head_camera_1, imu_1, lidar_1, wrist_camera_v1_1
+    drive:      wheel_{left,right}_1, {left,right}_motor_1, {left,right}_motor_mount_1
+    frames:     base_link, base_footprint, lidar_frame, imu_frame,
+                head_camera_frame, wrist_camera_frame
+  Visual origins are non-zero per-link: they are the mesh-centering offsets
+  for the Fusion-exported STLs (whose vertex data sits in a shared world frame
+  rooted at base_link).  See the canvas package for the derivation.
+  Kinematic tree:
+  - base_link
+     -[left_motor_mount_1_joint]-> left_motor_mount_1
+       -[left_motor_1_joint]-> left_motor_1
+         -[left_wheel_joint (continuous)]-> wheel_left_1
+     -[right_motor_mount_1_joint]-> right_motor_mount_1
+       -[right_motor_1_joint]-> right_motor_1
+         -[right_wheel_joint (continuous)]-> wheel_right_1
+     -[left_baseus_mount_v1_1_joint]-> left_baseus_mount_v1_1
+     -[frame_short_right_joint]-> frame_short_right
+     -[frame_tall_fr_joint]-> frame_tall_fr
+       -[frame_corner_fr_joint]-> frame_corner_fr
+     -[frame_tall_br_joint]-> frame_tall_br
+       -[modular_floor_joint]-> modular_floor
+         -[electronics_holder_left_joint]-> electronics_holder_left
+           -[electronics_pcb_joint]-> electronics_pcb
+             -[imu_1_joint]-> imu_1
+         -[electronics_holder_right_joint]-> electronics_holder_right
+       -[frame_corner_br_joint]-> frame_corner_br
+         -[frame_top_right_joint]-> frame_top_right
+     -[frame_tall_bl_joint]-> frame_tall_bl
+       -[frame_corner_bl_joint]-> frame_corner_bl
+         -[frame_top_back_joint]-> frame_top_back
+     -[frame_tall_fl_joint]-> frame_tall_fl
+       -[frame_corner_fl_joint]-> frame_corner_fl
+         -[frame_top_front_joint]-> frame_top_front
+           -[support_v1_1_joint]-> support_v1_1
+             -[tilt_servo_1_joint]-> tilt_servo_1
+               -[tilt (continuous)]-> realsense_support_v1_1
+                 -[head_camera_1_joint]-> head_camera_1
+         -[frame_top_left_joint]-> frame_top_left
+     -[frame_short_left_joint]-> frame_short_left
+       -[arm_deck_joint]-> arm_deck
+         -[arm_base_1_joint]-> arm_base_1
+           -[arm_base_rotation_servo_1_joint]-> arm_base_rotation_servo_1
+             -[1 (continuous)]-> arm_base_rotation_link_1
+               -[arm_shoulder_servo_1_joint]-> arm_shoulder_servo_1
+                 -[2 (continuous)]-> arm_shoulder_link_1
+                   -[arm_elbow_servo_1_joint]-> arm_elbow_servo_1
+                     -[3 (continuous)]-> arm_elbow_link_1
+                       -[arm_wrist_tilt_servo_1_joint]-> arm_wrist_tilt_servo_1
+                         -[4 (continuous)]-> arm_wrist_link_1
+                           -[arm_wrist_roll_servo_1_joint]-> arm_wrist_roll_servo_1
+                             -[5 (continuous)]-> arm_gripper_1
+                               -[arm_gripper_servo_1_joint]-> arm_gripper_servo_1
+                                 -[6 (continuous)]-> arm_jaw_1
+                               -[wrist_camera_mount_1_joint]-> wrist_camera_mount_1
+                                 -[wrist_camera_v1_1_joint]-> wrist_camera_v1_1
+               -[arm_base_rotation_link_cover_1_joint]-> arm_base_rotation_link_cover_1
+     -[right_caster_1_joint]-> right_caster_1
+     -[left_caster_1_joint]-> left_caster_1
+     -[llmy_lidar_base_v1_1_joint]-> llmy_lidar_base_v1_1
+       -[lidar_1_joint]-> lidar_1
+     -[right_baseus_mount_v1_1_joint]-> right_baseus_mount_v1_1
+-->
 <robot name="llmy_root" xmlns:xacro="http://www.ros.org/wiki/xacro">
-<!-- use_sim arg: set to false to exclude Gazebo sim hardware (for real robot) -->
-<xacro:arg name="use_sim" default="true"/>
-<xacro:include filename="$(find llmy_description)/urdf/materials.xacro" />
-<xacro:if value="$(arg use_sim)">
-  <xacro:include filename="$(find llmy_description)/urdf/LLMy.ros2control" />
-  <xacro:include filename="$(find llmy_description)/urdf/LLMy.gazebo" />
-</xacro:if>
-<!-- Base footprint for navigation -->
-<link name="base_footprint">
-</link>
-<joint name="base_footprint_joint" type="fixed">
-  <parent link="base_footprint"/>
-  <child link="base_link"/>
-  <origin xyz="0 0 0.015" rpy="0 0 0"/>
-</joint>
-<link name="base_link">
-  <inertial>
-    <origin xyz="-0.006203398028927208 4.883916027154101e-10 0.002469929870297714" rpy="0 0 0"/>
-    <mass value="1.569546654811132"/>
-    <inertia ixx="0.005179" iyy="0.005485" izz="0.010658" ixy="-0.0" iyz="-0.0" ixz="-3e-06"/>
-  </inertial>
-  <visual>
+  <!-- use_sim: when true, pulls in Gazebo ros2_control + sdf extensions.
+       Hardware launches should override to false. -->
+  <xacro:arg name="use_sim" default="true"/>
+  <xacro:include filename="$(find llmy_description)/urdf/materials.xacro" />
+  <xacro:if value="$(arg use_sim)">
+    <xacro:include filename="$(find llmy_description)/urdf/LLMy.ros2control" />
+    <xacro:include filename="$(find llmy_description)/urdf/LLMy.gazebo" />
+  </xacro:if>
+  <!-- ========================================== LINKS ==========================================-->
+  <link name="base_link">
+    <inertial>
+      <origin xyz="-0.003179 -0.000009 0.005401" rpy="0 0 0"/>
+      <mass value="2.227457140108448"/>
+      <inertia ixx="0.010888" iyy="0.009782" izz="0.020514" ixy="-5e-06" iyz="0.0" ixz="-3.3e-05"/>
+    </inertial>
+    <visual>
+      <origin xyz="0.000000 0.000000 0.000000" rpy="0 0 0"/>
+      <geometry><mesh filename="file://$(find llmy_description)/meshes/base_link.stl" scale="0.001 0.001 0.001"/></geometry>
+      <material name="nylon_darkgrey"/>
+    </visual>
+    <collision>
+      <origin xyz="0.000000 0.000000 0.000000" rpy="0 0 0"/>
+      <geometry><mesh filename="file://$(find llmy_description)/meshes/base_link.stl" scale="0.001 0.001 0.001"/></geometry>
+    </collision>
+  </link>
+  <link name="right_motor_mount_1">
+    <inertial>
+      <origin xyz="0.023782 0.003969 0.015577" rpy="0 0 0"/>
+      <mass value="0.19524814724461273"/>
+      <inertia ixx="4.7e-05" iyy="7.3e-05" izz="6.1e-05" ixy="-5e-06" iyz="5e-06" ixz="-1.5e-05"/>
+    </inertial>
+    <visual>
+      <origin xyz="-0.040000 0.080000 -0.005000" rpy="0 0 0"/>
+      <geometry><mesh filename="file://$(find llmy_description)/meshes/right_motor_mount_1.stl" scale="0.001 0.001 0.001"/></geometry>
+      <material name="metallic_green"/>
+    </visual>
+    <collision>
+      <origin xyz="-0.040000 0.080000 -0.005000" rpy="0 0 0"/>
+      <geometry><mesh filename="file://$(find llmy_description)/meshes/right_motor_mount_1.stl" scale="0.001 0.001 0.001"/></geometry>
+    </collision>
+  </link>
+  <link name="right_motor_1">
+    <inertial>
+      <origin xyz="-0.007742 -0.010688 -0.004446" rpy="0 0 0"/>
+      <mass value="0.06550661857714346"/>
+      <inertia ixx="4e-06" iyy="5e-06" izz="4e-06" ixy="0.0" iyz="-0.0" ixz="-0.0"/>
+    </inertial>
+    <visual>
+      <origin xyz="-0.067864 0.085855 -0.018700" rpy="0 0 0"/>
+      <geometry><mesh filename="file://$(find llmy_description)/meshes/wheel_right_in_1.stl" scale="0.001 0.001 0.001"/></geometry>
+      <material name="generic_grey"/>
+    </visual>
+    <collision>
+      <origin xyz="-0.067864 0.085855 -0.018700" rpy="0 0 0"/>
+      <geometry><mesh filename="file://$(find llmy_description)/meshes/wheel_right_in_1.stl" scale="0.001 0.001 0.001"/></geometry>
+    </collision>
+  </link>
+  <link name="wheel_right_1">
+    <inertial>
+      <origin xyz="-0.000000 0.003281 0.000000" rpy="0 0 0"/>
+      <mass value="0.47698614111454785"/>
+      <inertia ixx="0.000173" iyy="0.000323" izz="0.000173" ixy="0.0" iyz="0.0" ixz="0.0"/>
+    </inertial>
+    <visual>
+      <origin xyz="-0.060143 0.105270 -0.014242" rpy="0 0 0"/>
+      <geometry><mesh filename="file://$(find llmy_description)/meshes/wheel_right_out_1.stl" scale="0.001 0.001 0.001"/></geometry>
+      <material name="wheel_black"/>
+    </visual>
+    <collision>
+      <origin xyz="-0.060143 0.105270 -0.014242" rpy="0 0 0"/>
+      <geometry><mesh filename="file://$(find llmy_description)/meshes/wheel_right_out_1.stl" scale="0.001 0.001 0.001"/></geometry>
+    </collision>
+  </link>
+  <link name="left_motor_mount_1">
+    <inertial>
+      <origin xyz="0.023783 -0.003969 0.015577" rpy="0 0 0"/>
+      <mass value="0.19524842528531677"/>
+      <inertia ixx="4.7e-05" iyy="7.3e-05" izz="6.1e-05" ixy="5e-06" iyz="-5e-06" ixz="-1.5e-05"/>
+    </inertial>
+    <visual>
+      <origin xyz="-0.040000 -0.080000 -0.005000" rpy="0 0 0"/>
+      <geometry><mesh filename="file://$(find llmy_description)/meshes/left_motor_mount_1.stl" scale="0.001 0.001 0.001"/></geometry>
+      <material name="metallic_green"/>
+    </visual>
+    <collision>
+      <origin xyz="-0.040000 -0.080000 -0.005000" rpy="0 0 0"/>
+      <geometry><mesh filename="file://$(find llmy_description)/meshes/left_motor_mount_1.stl" scale="0.001 0.001 0.001"/></geometry>
+    </collision>
+  </link>
+  <link name="left_motor_1">
+    <inertial>
+      <origin xyz="0.007701 0.010688 -0.004446" rpy="0 0 0"/>
+      <mass value="0.06550661857714346"/>
+      <inertia ixx="4e-06" iyy="5e-06" izz="4e-06" ixy="-0.0" iyz="0.0" ixz="-0.0"/>
+    </inertial>
+    <visual>
+      <origin xyz="-0.052275 -0.085855 -0.018700" rpy="0 0 0"/>
+      <geometry><mesh filename="file://$(find llmy_description)/meshes/wheel_left_in_1.stl" scale="0.001 0.001 0.001"/></geometry>
+      <material name="generic_grey"/>
+    </visual>
+    <collision>
+      <origin xyz="-0.052275 -0.085855 -0.018700" rpy="0 0 0"/>
+      <geometry><mesh filename="file://$(find llmy_description)/meshes/wheel_left_in_1.stl" scale="0.001 0.001 0.001"/></geometry>
+    </collision>
+  </link>
+  <link name="wheel_left_1">
+    <inertial>
+      <origin xyz="0.000000 -0.003281 0.000000" rpy="0 0 0"/>
+      <mass value="0.47698614111454785"/>
+      <inertia ixx="0.000173" iyy="0.000323" izz="0.000173" ixy="-0.0" iyz="0.0" ixz="0.0"/>
+    </inertial>
+    <visual>
+      <origin xyz="-0.059996 -0.105270 -0.014242" rpy="0 0 0"/>
+      <geometry><mesh filename="file://$(find llmy_description)/meshes/wheel_left_out_1.stl" scale="0.001 0.001 0.001"/></geometry>
+      <material name="wheel_black"/>
+    </visual>
+    <collision>
+      <origin xyz="-0.059996 -0.105270 -0.014242" rpy="0 0 0"/>
+      <geometry><mesh filename="file://$(find llmy_description)/meshes/wheel_left_out_1.stl" scale="0.001 0.001 0.001"/></geometry>
+    </collision>
+  </link>
+  <link name="right_caster_1">
+    <inertial>
+      <origin xyz="-0.000000 0.007747 -0.008951" rpy="0 0 0"/>
+      <mass value="0.04903387471960177"/>
+      <inertia ixx="3e-06" iyy="3e-06" izz="3e-06" ixy="-0.0" iyz="0.0" ixz="0.0"/>
+    </inertial>
+    <visual>
+      <origin xyz="0.080000 -0.072253 0.000000" rpy="0 0 0"/>
+      <geometry><mesh filename="file://$(find llmy_description)/meshes/right_caster_1.stl" scale="0.001 0.001 0.001"/></geometry>
+      <material name="caster_blue"/>
+    </visual>
+    <collision>
+      <origin xyz="0.080000 -0.072253 0.000000" rpy="0 0 0"/>
+      <geometry><mesh filename="file://$(find llmy_description)/meshes/right_caster_1.stl" scale="0.001 0.001 0.001"/></geometry>
+    </collision>
+  </link>
+  <link name="left_caster_1">
+    <inertial>
+      <origin xyz="-0.000000 -0.007747 -0.008951" rpy="0 0 0"/>
+      <mass value="0.04903387471960177"/>
+      <inertia ixx="3e-06" iyy="3e-06" izz="3e-06" ixy="-0.0" iyz="0.0" ixz="0.0"/>
+    </inertial>
+    <visual>
+      <origin xyz="0.080000 0.072253 0.000000" rpy="0 0 0"/>
+      <geometry><mesh filename="file://$(find llmy_description)/meshes/left_caster_1.stl" scale="0.001 0.001 0.001"/></geometry>
+      <material name="caster_blue"/>
+    </visual>
+    <collision>
+      <origin xyz="0.080000 0.072253 0.000000" rpy="0 0 0"/>
+      <geometry><mesh filename="file://$(find llmy_description)/meshes/left_caster_1.stl" scale="0.001 0.001 0.001"/></geometry>
+    </collision>
+  </link>
+  <link name="right_baseus_mount_v1_1">
+    <inertial>
+      <origin xyz="0.019691 -0.001860 0.023385" rpy="0 0 0"/>
+      <mass value="0.0655308096957003"/>
+      <inertia ixx="3.1e-05" iyy="5.4e-05" izz="2.4e-05" ixy="0.0" iyz="1e-06" ixz="-0.0"/>
+    </inertial>
+    <visual>
+      <origin xyz="0.060000 -0.080000 -0.005000" rpy="0 0 0"/>
+      <geometry><mesh filename="file://$(find llmy_description)/meshes/right_battery_mount_1.stl" scale="0.001 0.001 0.001"/></geometry>
+      <material name="metallic_green"/>
+    </visual>
+    <collision>
+      <origin xyz="0.060000 -0.080000 -0.005000" rpy="0 0 0"/>
+      <geometry><mesh filename="file://$(find llmy_description)/meshes/right_battery_mount_1.stl" scale="0.001 0.001 0.001"/></geometry>
+    </collision>
+  </link>
+  <link name="left_baseus_mount_v1_1">
+    <inertial>
+      <origin xyz="0.019691 0.001860 0.023385" rpy="0 0 0"/>
+      <mass value="0.06553077893811926"/>
+      <inertia ixx="3.1e-05" iyy="5.4e-05" izz="2.4e-05" ixy="-0.0" iyz="-1e-06" ixz="-0.0"/>
+    </inertial>
+    <visual>
+      <origin xyz="0.060000 0.080000 -0.005000" rpy="0 0 0"/>
+      <geometry><mesh filename="file://$(find llmy_description)/meshes/left_battery_mount_1.stl" scale="0.001 0.001 0.001"/></geometry>
+      <material name="metallic_green"/>
+    </visual>
+    <collision>
+      <origin xyz="0.060000 0.080000 -0.005000" rpy="0 0 0"/>
+      <geometry><mesh filename="file://$(find llmy_description)/meshes/left_battery_mount_1.stl" scale="0.001 0.001 0.001"/></geometry>
+    </collision>
+  </link>
+  <link name="llmy_lidar_base_v1_1">
+    <inertial>
+      <origin xyz="0.015962 -0.073645 -0.015094" rpy="0 0 0"/>
+      <mass value="0.3979913592232491"/>
+      <inertia ixx="0.001129" iyy="6.9e-05" izz="0.001183" ixy="-0.0" iyz="-0.0" ixz="6e-06"/>
+    </inertial>
+    <visual>
+      <origin xyz="-0.110000 -0.073755 -0.020000" rpy="0 0 0"/>
+      <geometry><mesh filename="file://$(find llmy_description)/meshes/lidar_mount_1.stl" scale="0.001 0.001 0.001"/></geometry>
+      <material name="metallic_green"/>
+    </visual>
+    <collision>
+      <origin xyz="-0.110000 -0.073755 -0.020000" rpy="0 0 0"/>
+      <geometry><mesh filename="file://$(find llmy_description)/meshes/lidar_mount_1.stl" scale="0.001 0.001 0.001"/></geometry>
+    </collision>
+  </link>
+  <link name="lidar_1">
+    <inertial>
+      <origin xyz="-0.021415 -0.021595 0.014018" rpy="0 0 0"/>
+      <mass value="0.2536750002862165"/>
+      <inertia ixx="0.000111" iyy="0.000111" izz="0.000157" ixy="-0.0" iyz="-0.0" ixz="0.0"/>
+    </inertial>
+    <visual>
+      <origin xyz="-0.145700 -0.023250 -0.008000" rpy="0 0 0"/>
+      <geometry><mesh filename="file://$(find llmy_description)/meshes/lidar_1.stl" scale="0.001 0.001 0.001"/></geometry>
+      <material name="epx_darkgrey"/>
+    </visual>
+    <collision>
+      <origin xyz="-0.145700 -0.023250 -0.008000" rpy="0 0 0"/>
+      <geometry><mesh filename="file://$(find llmy_description)/meshes/lidar_1.stl" scale="0.001 0.001 0.001"/></geometry>
+    </collision>
+  </link>
+  <link name="frame_short_right">
+    <inertial>
+      <origin xyz="-0.000000 0.000000 0.037500" rpy="0 0 0"/>
+      <mass value="0.10216504467841848"/>
+      <inertia ixx="5.2e-05" iyy="5.2e-05" izz="9e-06" ixy="-0.0" iyz="-0.0" ixz="-0.0"/>
+    </inertial>
+    <visual>
+      <origin xyz="-0.095000 0.073755 -0.005000" rpy="0 0 0"/>
+      <geometry><mesh filename="file://$(find llmy_description)/meshes/short_2020_1.stl" scale="0.001 0.001 0.001"/></geometry>
+      <material name="aluminum_polished"/>
+    </visual>
+    <collision>
+      <origin xyz="-0.095000 0.073755 -0.005000" rpy="0 0 0"/>
+      <geometry><mesh filename="file://$(find llmy_description)/meshes/short_2020_1.stl" scale="0.001 0.001 0.001"/></geometry>
+    </collision>
+  </link>
+  <link name="frame_short_left">
+    <inertial>
+      <origin xyz="-0.000000 -0.000000 0.037500" rpy="0 0 0"/>
+      <mass value="0.10216504467841848"/>
+      <inertia ixx="5.2e-05" iyy="5.2e-05" izz="9e-06" ixy="-0.0" iyz="-0.0" ixz="-0.0"/>
+    </inertial>
+    <visual>
+      <origin xyz="-0.095000 -0.073755 -0.005000" rpy="0 0 0"/>
+      <geometry><mesh filename="file://$(find llmy_description)/meshes/short_2020__1__1.stl" scale="0.001 0.001 0.001"/></geometry>
+      <material name="aluminum_polished"/>
+    </visual>
+    <collision>
+      <origin xyz="-0.095000 -0.073755 -0.005000" rpy="0 0 0"/>
+      <geometry><mesh filename="file://$(find llmy_description)/meshes/short_2020__1__1.stl" scale="0.001 0.001 0.001"/></geometry>
+    </collision>
+  </link>
+  <link name="frame_tall_bl">
+    <inertial>
+      <origin xyz="-0.000016 0.000013 0.001354" rpy="0 0 0"/>
+      <mass value="0.4366746675159977"/>
+      <inertia ixx="0.003758" iyy="0.003758" izz="3.7e-05" ixy="-0.0" iyz="-0.0" ixz="-0.0"/>
+    </inertial>
+    <visual>
+      <origin xyz="0.094984 -0.099987 -0.163929" rpy="0 0 0"/>
+      <geometry><mesh filename="file://$(find llmy_description)/meshes/tall_2020_1.stl" scale="0.001 0.001 0.001"/></geometry>
+      <material name="aluminum_polished"/>
+    </visual>
+    <collision>
+      <origin xyz="0.094984 -0.099987 -0.163929" rpy="0 0 0"/>
+      <geometry><mesh filename="file://$(find llmy_description)/meshes/tall_2020_1.stl" scale="0.001 0.001 0.001"/></geometry>
+    </collision>
+  </link>
+  <link name="frame_tall_br">
+    <inertial>
+      <origin xyz="-0.000016 0.000013 0.001354" rpy="0 0 0"/>
+      <mass value="0.4366746675159977"/>
+      <inertia ixx="0.003758" iyy="0.003758" izz="3.7e-05" ixy="-0.0" iyz="-0.0" ixz="-0.0"/>
+    </inertial>
+    <visual>
+      <origin xyz="0.094984 0.100013 -0.163929" rpy="0 0 0"/>
+      <geometry><mesh filename="file://$(find llmy_description)/meshes/tall_2020_2.stl" scale="0.001 0.001 0.001"/></geometry>
+      <material name="aluminum_polished"/>
+    </visual>
+    <collision>
+      <origin xyz="0.094984 0.100013 -0.163929" rpy="0 0 0"/>
+      <geometry><mesh filename="file://$(find llmy_description)/meshes/tall_2020_2.stl" scale="0.001 0.001 0.001"/></geometry>
+    </collision>
+  </link>
+  <link name="frame_tall_fr">
+    <inertial>
+      <origin xyz="-0.000016 0.000013 0.001354" rpy="0 0 0"/>
+      <mass value="0.4366746675159977"/>
+      <inertia ixx="0.003758" iyy="0.003758" izz="3.7e-05" ixy="-0.0" iyz="-0.0" ixz="-0.0"/>
+    </inertial>
+    <visual>
+      <origin xyz="-0.005005 0.100013 -0.163929" rpy="0 0 0"/>
+      <geometry><mesh filename="file://$(find llmy_description)/meshes/tall_2020_3.stl" scale="0.001 0.001 0.001"/></geometry>
+      <material name="aluminum_polished"/>
+    </visual>
+    <collision>
+      <origin xyz="-0.005005 0.100013 -0.163929" rpy="0 0 0"/>
+      <geometry><mesh filename="file://$(find llmy_description)/meshes/tall_2020_3.stl" scale="0.001 0.001 0.001"/></geometry>
+    </collision>
+  </link>
+  <link name="frame_tall_fl">
+    <inertial>
+      <origin xyz="-0.000016 0.000013 0.001354" rpy="0 0 0"/>
+      <mass value="0.4366746675159977"/>
+      <inertia ixx="0.003758" iyy="0.003758" izz="3.7e-05" ixy="-0.0" iyz="-0.0" ixz="-0.0"/>
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
File: ros/src/llmy_description/urdf/materials.xacro (robot description, xacro)
@@ -1,6 +1,43 @@
 <?xml version="1.0" ?>
-<robot name="llmy_root" xmlns:xacro="http://www.ros.org/wiki/xacro" >
-<material name="silver">
-  <color rgba="0.700 0.700 0.700 1.000"/>
-</material>
+<robot name="llmy_canvas" xmlns:xacro="http://www.ros.org/wiki/xacro">
+  <!-- EPX 150 - Air Baked composite (structural arm links, decks, lidar housing). -->
+  <material name="epx_darkgrey">
+    <color rgba="0.200 0.200 0.200 1.0"/>
+  </material>
+  <!-- PA 12 - Nylon - PA 603-CF (carbon-filled nylon, e.g. base_link, wrist camera body). -->
+  <material name="nylon_darkgrey">
+    <color rgba="0.180 0.180 0.200 1.0"/>
+  </material>
+  <!-- Steel - Satin (SO-101 servo housings, camera tilt servo). -->
+  <material name="steel_satin">
+    <color rgba="0.620 0.630 0.660 1.0"/>
+  </material>
+  <!-- Aluminum - Polished (2020 extrusions, head camera body). -->
+  <material name="aluminum_polished">
+    <color rgba="0.850 0.870 0.900 1.0"/>
+  </material>
+  <!-- Paint - Metallic Green (3-way corners, mounts, camera holder, waist cover). -->
+  <material name="metallic_green">
+    <color rgba="0.102 0.345 0.176 1.0"/>
+  </material>
+  <!-- Pure green (battery mounts, RGB 0,128,0). -->
+  <material name="pure_green">
+    <color rgba="0.000 0.502 0.000 1.0"/>
+  </material>
+  <!-- Near-black wheel tires (RGB 25,25,25). -->
+  <material name="wheel_black">
+    <color rgba="0.098 0.098 0.098 1.0"/>
+  </material>
+  <!-- Light blue casters (RGB 202,209,238). -->
+  <material name="caster_blue">
+    <color rgba="0.792 0.820 0.933 1.0"/>
+  </material>
+  <!-- Generic placeholder for Fusion "Generic" material (PCB, wheel hubs, etc.). -->
+  <material name="generic_grey">
+    <color rgba="0.550 0.550 0.550 1.0"/>
+  </material>
+  <!-- Legacy name retained for compatibility. -->
+  <material name="silver">
+    <color rgba="0.700 0.700 0.700 1.0"/>
+  </material>
 </robot>
